File: keyboard.kicad_pcb (KiCad board)
At the start: 2 copper layers, 357.7 x 105.2 mm, 159 parts, among them SW1 SW_PUSH, U2 ATMEGA32U4, X2 XTAL_GND

Commit message: Testing
Parts:
- moved U2 48.9 mm to (341.6, 47.0)
