File: keyboard.sch (KiCad schematic (older format))
At the start: 149 parts, among them J1 USB_mini_micro_B, U1 ATMEGA32U4

Commit message: Testing
Parts:
- removed R3, R4: 22, Resistor_SMD:R_0805_2012Metric_Pad1.15x1.40mm_HandSolder, symbol Device:R
- added R3 (x2): 22, Resistor_SMD:R_0805_2012Metric_Pad1.15x1.40mm_HandSolder, symbol Device:R
